File: wing.sch (KiCad schematic (older format))
At the start: 55 parts, among them J1 pin_array_2x1, U1 DSP310_DEV, U10 DSP310_DEV, U11 DSP310_DEV, U12 DSP310_DEV, U13 DSP310_DEV, U14 DSP310_DEV, U15 DSP310_DEV, U16 DSP310_DEV, U17 DSP310_DEV, U18 DSP310_DEV, U19 DSP310_DEV, U2 DSP310_DEV, U20 DSP310_DEV, U21 DSP310_DEV, U22 DSP310_DEV, U23 DSP310_DEV, U24 DSP310_DEV, U25 DSP310_DEV, U26 DSP310_DEV, U27 DSP310_DEV, U28 DSP310_DEV, U29 DSP310_DEV, U3 DSP310_DEV, U30 DSP310_DEV, U31 DSP310_DEV, U32 DSP310_DEV, U33 DSP310_DEV, U34 DSP310_DEV, U35 DSP310_DEV, U36 DSP310_DEV, U37 DSP310_DEV, U38 DSP310_DEV, U39 DSP310_DEV, U4 DSP310_DEV, U40 DSP310_DEV, U41 DSP310_DEV, U42 DSP310_DEV, U43 DSP310_DEV, U44 DSP310_DEV, U45 DSP310_DEV, U46 DSP310_DEV, U47 DSP310_DEV, U48 DSP310_DEV, U49 DSP310_DEV, U5 DSP310_DEV, U50 DSP310_DEV, U51 DSP310_DEV, U52 DSP310_DEV, U54 Adafruit_BNO055, U6 DSP310_DEV, U7 DSP310_DEV, U8 DSP310_DEV, U9 DSP310_DEV

Commit message: Finished initial schematic, footprint design and footprint assignment.
Parts:
- J1: footprint (none) -> JST_PH_2PIN:JST_PH_2PIN
- U1, U2: footprint (none) -> dps310_dev:DPS310_DEV
- U10, U11, U12, U13, U14, U15, U16, U17, U18, U19, U20, U21, U22, U23, U24, U25, U26, U27, U28, U29, U3, U30, U31, U32, U33, U34, U35, U36, U37, U38, U39, U4, U40, U41, U42, U43, U44, U45, U46, U47, U48, U49, U5, U50, U51, U52, U6, U7, U8, U9: value DSP310_DEV -> DPS310_DEV; footprint (none) -> dps310_dev:DPS310_DEV
- U53: renamed from U?; footprint (none) -> teensy35:teensy3.5
- U54: footprint (none) -> Adafruit_BNO055:Adafruit_BNO055
Connections:
- net DSP_CS00 is gone; now on net DPS_CS00: U1.6 (CSB)
- net DSP_CS01 is gone; now on net DPS_CS01: U2.6 (CSB)
- net DSP_CS02 is gone; now on net DPS_CS02: U3.6 (CSB)
- net DSP_CS03 is gone; now on net DPS_CS03: U4.6 (CSB)
- net DSP_CS04 is gone; now on net DPS_CS04: U5.6 (CSB)
- net DSP_CS05 is gone; now on net DPS_CS05: U6.6 (CSB)
- net DSP_CS06 is gone; now on net DPS_CS06: U7.6 (CSB)
- net DSP_CS07 is gone; now on net DPS_CS07: U8.6 (CSB)
- net DSP_CS08 is gone; now on net DPS_CS08: U9.6 (CSB)
- net DSP_CS09 is gone; now on net DPS_CS09: U10.6 (CSB)
- net DSP_CS10 is gone; now on net DPS_CS10: U11.6 (CSB)
- net DSP_CS11 is gone; now on net DPS_CS11: U12.6 (CSB)
- net DSP_CS12 is gone; now on net DPS_CS12: U13.6 (CSB)
- net DSP_CS13 is gone; now on net DPS_CS13: U14.6 (CSB)
- net DSP_CS14 is gone; now on net DPS_CS14: U15.6 (CSB)
- net DSP_CS15 is gone; now on net DPS_CS15: U16.6 (CSB)
- net DSP_CS16 is gone; now on net DPS_CS16: U17.6 (CSB)
- net DSP_CS17 is gone; now on net DPS_CS17: U18.6 (CSB)
- net DSP_CS18 is gone; now on net DPS_CS18: U19.6 (CSB)
- net DSP_CS19 is gone; now on net DPS_CS19: U20.6 (CSB)
- net DSP_CS20 is gone; now on net DPS_CS20: U21.6 (CSB)
- net DSP_CS21 is gone; now on net DPS_CS21: U22.6 (CSB)
- net DSP_CS22 is gone; now on net DPS_CS22: U23.6 (CSB)
- net DSP_CS23 is gone; now on net DPS_CS23: U24.6 (CSB)
- net DSP_CS24 is gone; now on net DPS_CS24: U25.6 (CSB)
- net DSP_CS25 is gone; now on net DPS_CS25: U26.6 (CSB)
- net DSP_CS26 is gone; now on net DPS_CS26: U27.6 (CSB)
- net DSP_CS27 is gone; now on net DPS_CS27: U28.6 (CSB)
- net DSP_CS28 is gone; now on net DPS_CS28: U29.6 (CSB)
- net DSP_CS29 is gone; now on net DPS_CS29: U30.6 (CSB)
- net DSP_CS30 is gone; now on net DPS_CS30: U31.6 (CSB)
- net DSP_CS31 is gone; now on net DPS_CS31: U32.6 (CSB)
- net DSP_CS32 is gone; now on net DPS_CS32: U33.6 (CSB)
- net DSP_CS33 is gone; now on net DPS_CS33: U34.6 (CSB)
- net DSP_CS34 is gone; now on net DPS_CS34: U35.6 (CSB)
- net DSP_CS35 is gone; now on net DPS_CS35: U36.6 (CSB)
- net DSP_CS36 is gone; now on net DPS_CS36: U37.6 (CSB)
- net DSP_CS37 is gone; now on net DPS_CS37: U38.6 (CSB)
- net DSP_CS38 is gone; now on net DPS_CS38: U39.6 (CSB)
- net DSP_CS39 is gone; now on net DPS_CS39: U40.6 (CSB)
- net DSP_CS40 is gone; now on net DPS_CS40: U41.6 (CSB)
- net DSP_CS41 is gone; now on net DPS_CS41: U42.6 (CSB)
- net DSP_CS42 is gone; now on net DPS_CS42: U43.6 (CSB)
- net DSP_CS43 is gone; now on net DPS_CS43: U44.6 (CSB)
- net DSP_CS44 is gone; now on net DPS_CS44: U45.6 (CSB)
- net DSP_CS45 is gone; now on net DPS_CS45: U46.6 (CSB)
- net DSP_CS46 is gone; now on net DPS_CS46: U47.6 (CSB)
- net DSP_CS47 is gone; now on net DPS_CS47: U48.6 (CSB)
- net DSP_CS48 is gone; now on net DPS_CS48: U49.6 (CSB)
- net DSP_CS49 is gone; now on net DPS_CS49: U50.6 (CSB)
- net DSP_CS50 is gone; now on net DPS_CS50: U51.6 (CSB)
- net DSP_CS51 is gone; now on net DPS_CS51: U52.6 (CSB)
- net GND: now also U53.34 (GND)
- net DPS_CS3 renamed DPS_CS03
- net DPS_CS4 renamed DPS_CS04
- net DPS_CS5 renamed DPS_CS05
- net DPS_CS6 renamed DPS_CS06
- net DPS_CS7 renamed DPS_CS07
- net DPS_CS8 renamed DPS_CS08
- net DPS_CS9 renamed DPS_CS09
- no-connect marks 84 -> 78
Other:
- note added: "JST PH SERIES \nDIGIKEY PN 455-1719-ND \nSPARKFUN PN PRT-09749\n"
- moved on the sheet: J1, U54
