File: wing.kicad_pcb (KiCad board)
At the start: 2 copper layers, 0 parts

Commit message: Finished initial schematic, footprint design and footprint assignment.
Parts:
- added J1: pin_array_2x1, JST_PH_2PIN:JST_PH_2PIN, F.Cu at (172.3, -147.5)
- added U1: DSP310_DEV, dps310_dev:DPS310_DEV, F.Cu at (55.0, -148.8)
- added U10: DPS310_DEV, dps310_dev:DPS310_DEV, F.Cu at (55.0, -122.5)
- added U11: DPS310_DEV, dps310_dev:DPS310_DEV, F.Cu at (72.4, -122.5)
- added U12: DPS310_DEV, dps310_dev:DPS310_DEV, F.Cu at (37.6, -148.8)
- added U13: DPS310_DEV, dps310_dev:DPS310_DEV, F.Cu at (55.0, -109.3)
- added U14: DPS310_DEV, dps310_dev:DPS310_DEV, F.Cu at (142.0, -122.5)
- added U15: DPS310_DEV, dps310_dev:DPS310_DEV, F.Cu at (40.1, -96.2)
- added U16: DPS310_DEV, dps310_dev:DPS310_DEV, F.Cu at (57.5, -96.2)
- added U17: DPS310_DEV, dps310_dev:DPS310_DEV, F.Cu at (40.1, -83.0)
- added U18: DPS310_DEV, dps310_dev:DPS310_DEV, F.Cu at (107.2, -135.6)
- added U19: DPS310_DEV, dps310_dev:DPS310_DEV, F.Cu at (40.1, -69.9)
- added U2: DSP310_DEV, dps310_dev:DPS310_DEV, F.Cu at (72.4, -148.8)
- added U20: DPS310_DEV, dps310_dev:DPS310_DEV, F.Cu at (72.4, -109.3)
- added U21: DPS310_DEV, dps310_dev:DPS310_DEV, F.Cu at (89.8, -122.5)
- added U22: DPS310_DEV, dps310_dev:DPS310_DEV, F.Cu at (124.6, -148.8)
- added U23: DPS310_DEV, dps310_dev:DPS310_DEV, F.Cu at (57.5, -83.0)
- added U24: DPS310_DEV, dps310_dev:DPS310_DEV, F.Cu at (74.9, -96.2)
- added U25: DPS310_DEV, dps310_dev:DPS310_DEV, F.Cu at (107.2, -122.5)
- added U26: DPS310_DEV, dps310_dev:DPS310_DEV, F.Cu at (37.6, -109.3)
- added U27: DPS310_DEV, dps310_dev:DPS310_DEV, F.Cu at (159.4, -135.6)
- added U28: DPS310_DEV, dps310_dev:DPS310_DEV, F.Cu at (57.5, -69.9)
- added U29: DPS310_DEV, dps310_dev:DPS310_DEV, F.Cu at (142.0, -148.8)
- added U3: DPS310_DEV, dps310_dev:DPS310_DEV, F.Cu at (89.8, -148.8)
- added U30: DPS310_DEV, dps310_dev:DPS310_DEV, F.Cu at (74.9, -83.0)
- added U31: DPS310_DEV, dps310_dev:DPS310_DEV, F.Cu at (92.3, -96.2)
- added U32: DPS310_DEV, dps310_dev:DPS310_DEV, F.Cu at (107.2, -109.3)
- added U33: DPS310_DEV, dps310_dev:DPS310_DEV, F.Cu at (124.6, -122.5)
- added U34: DPS310_DEV, dps310_dev:DPS310_DEV, F.Cu at (142.0, -135.6)
- added U35: DPS310_DEV, dps310_dev:DPS310_DEV, F.Cu at (74.9, -69.9)
- added U36: DPS310_DEV, dps310_dev:DPS310_DEV, F.Cu at (159.4, -148.8)
- added U37: DPS310_DEV, dps310_dev:DPS310_DEV, F.Cu at (92.3, -83.0)
- added U38: DPS310_DEV, dps310_dev:DPS310_DEV, F.Cu at (109.7, -96.2)
- added U39: DPS310_DEV, dps310_dev:DPS310_DEV, F.Cu at (124.6, -109.3)
- added U4: DPS310_DEV, dps310_dev:DPS310_DEV, F.Cu at (107.2, -148.8)
- added U40: DPS310_DEV, dps310_dev:DPS310_DEV, F.Cu at (124.6, -135.6)
- added U41: DPS310_DEV, dps310_dev:DPS310_DEV, F.Cu at (89.8, -109.3)
- added U42: DPS310_DEV, dps310_dev:DPS310_DEV, F.Cu at (92.3, -69.9)
- added U43: DPS310_DEV, dps310_dev:DPS310_DEV, F.Cu at (109.7, -83.0)
- added U44: DPS310_DEV, dps310_dev:DPS310_DEV, F.Cu at (127.1, -96.2)
- added U45: DPS310_DEV, dps310_dev:DPS310_DEV, F.Cu at (142.0, -109.3)
- added U46: DPS310_DEV, dps310_dev:DPS310_DEV, F.Cu at (159.4, -122.5)
- added U47: DPS310_DEV, dps310_dev:DPS310_DEV, F.Cu at (109.7, -69.9)
- added U48: DPS310_DEV, dps310_dev:DPS310_DEV, F.Cu at (127.1, -83.0)
- added U49: DPS310_DEV, dps310_dev:DPS310_DEV, F.Cu at (144.6, -96.2)
- added U5: DPS310_DEV, dps310_dev:DPS310_DEV, F.Cu at (37.6, -135.6)
- added U50: DPS310_DEV, dps310_dev:DPS310_DEV, F.Cu at (159.4, -109.3)
- added U51: DPS310_DEV, dps310_dev:DPS310_DEV, F.Cu at (127.1, -69.9)
- added U52: DPS310_DEV, dps310_dev:DPS310_DEV, F.Cu at (144.6, -83.0)
- added U53: teensy3.5, teensy35:teensy3.5, F.Cu at (19.6, -122.6)
- added U54: Adafruit_BNO055, Adafruit_BNO055:Adafruit_BNO055, F.Cu at (20.9, -76.9)
- added U6: DPS310_DEV, dps310_dev:DPS310_DEV, F.Cu at (55.0, -135.6)
- added U7: DPS310_DEV, dps310_dev:DPS310_DEV, F.Cu at (72.4, -135.6)
- added U8: DPS310_DEV, dps310_dev:DPS310_DEV, F.Cu at (89.8, -135.6)
- added U9: DPS310_DEV, dps310_dev:DPS310_DEV, F.Cu at (37.6, -122.5)

Commit message: Finished initial design.  Needs to be routed.
Parts:
- added H1: cable_tie_hole, cable_tie_hole:cable_tie_hole, F.Cu at (214.0, 104.0)
- added H2: cable_tie_hole, cable_tie_hole:cable_tie_hole, F.Cu at (224.0, 104.0)
- added H3: cable_tie_hole, cable_tie_hole:cable_tie_hole, F.Cu at (214.0, 118.0)
- added H4: cable_tie_hole, cable_tie_hole:cable_tie_hole, F.Cu at (224.0, 118.0)
- added H5: cable_tie_hole, cable_tie_hole:cable_tie_hole, F.Cu at (224.0, 123.0)
- added H6: cable_tie_hole, cable_tie_hole:cable_tie_hole, F.Cu at (224.0, 128.0)
- U27, U28, U29, U30, U31, U32, U33, U34, U35, U36, U37, U38, U39, U40, U41, U42, U43, U44, U45, U46, U47, U48, U49, U50, U51, U52: moved to B.Cu
- moved U26 284.9 mm to (182.4, 136.0), turned to 180 degrees
- moved U53 278.9 mm to (171.6, 111.2), turned to 270 degrees
- moved J1 274.6 mm to (206.0, 125.0), turned to 270 degrees
- moved U18 261.2 mm to (122.4, 125.1), turned to 180 degrees
- moved U21 257.2 mm to (142.4, 129.3), turned to 180 degrees
- moved U4 251.1 mm to (66.2, 98.9), turned to 180 degrees
- moved U24 245.4 mm to (162.4, 133.0), turned to 180 degrees
- moved U27 242.6 mm to (51.6, 81.7), turned to 270 degrees
- moved U50 242.4 mm to (162.4, 133.0)
- moved U40 241.8 mm to (102.3, 105.1), turned to 180 degrees
- moved U29 241.4 mm to (66.2, 80.4), turned to 180 degrees
- moved U34 239.4 mm to (84.2, 96.7), turned to 180 degrees
- moved U9 238.5 mm to (84.3, 111.4), turned to 180 degrees
- moved U54 236.0 mm to (189.5, 88.1), turned to 90 degrees
- moved U12 234.6 mm to (102.2, 76.7)
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Other:
- board outline added: 198.4 x 102.7 mm
- board text added: "GND"
- board text added: "Robofly DPS310 Wing V0.1 Dickinson Lab 2019"
- board text added: "SYNC"

Commit message: Added readme and images.
Routing:
- net /3V3: track 0.00 -> 1084.0 mm, vias 0 -> 15
- net GND: track 0.00 -> 865.0 mm, vias 0 -> 19
- net /MISO: track 0.00 -> 846.5 mm, vias 0 -> 17
- net /SCK: track 0.00 -> 759.1 mm, vias 0 -> 18
- net /MOSI: track 0.00 -> 679.5 mm, vias 0 -> 24
- net /DPS_CS00: track 0.00 -> 170.3 mm, vias 0 -> 1
- net /DPS_CS01: track 0.00 -> 157.9 mm, vias 0 -> 1
- net /DPS_CS15: track 0.00 -> 154.6 mm, vias 0 -> 1
- net /DPS_CS44: track 0.00 -> 152.6 mm, vias 0 -> 1
- net /DPS_CS43: track 0.00 -> 151.4 mm, vias 0 -> 1
- net /DPS_CS42: track 0.00 -> 150.3 mm, vias 0 -> 1
- net /DPS_CS47: track 0.00 -> 143.8 mm, vias 0 -> 1
- net /DPS_CS03: track 0.00 -> 138.4 mm
- net /DPS_CS16: track 0.00 -> 136.4 mm, vias 0 -> 2
- net /DPS_CS46: track 0.00 -> 135.7 mm, vias 0 -> 2
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